File: Fuji-Synth/Fuji-Synth.kicad_sch (KiCad schematic)
At the start: 54 parts, among them J1 AudioJack3, SW1 SW_Push, SW2 SW_Push, SW3 RotaryEncoder_Switch, SW4 RotaryEncoder_Switch, SW5 RotaryEncoder_Switch, U1 MPR121QR2, U2 PCM5102A, U3 ER_OLEDM0.91_1x-I2C

Commit message: Finished with Schematic v1.0 / Added footprints / Created footprint for test points
Parts:
- A1: footprint Module:RaspberryPi_Pico_Common_Unspecified -> Module:RaspberryPi_Pico_Common_THT
- C1: renamed from C6; footprint (none) -> Capacitor_SMD:C_0805_2012Metric_Pad1.18x1.45mm_HandSolder
- C10: renamed from C3; footprint (none) -> Capacitor_SMD:C_0805_2012Metric_Pad1.18x1.45mm_HandSolder
- C11, C12: footprint (none) -> Capacitor_SMD:C_0805_2012Metric_Pad1.18x1.45mm_HandSolder
- C2: renamed from C4; footprint (none) -> Capacitor_SMD:C_0805_2012Metric_Pad1.18x1.45mm_HandSolder
- C3: renamed from C5; footprint (none) -> Capacitor_SMD:C_0805_2012Metric_Pad1.18x1.45mm_HandSolder
- C4: renamed from C8; footprint (none) -> Capacitor_SMD:C_0805_2012Metric_Pad1.18x1.45mm_HandSolder
- C5: renamed from C7; footprint (none) -> Capacitor_SMD:C_0805_2012Metric_Pad1.18x1.45mm_HandSolder
- C6: renamed from C9; footprint (none) -> Capacitor_SMD:C_0805_2012Metric_Pad1.18x1.45mm_HandSolder
- C7: renamed from C1; footprint (none) -> Capacitor_SMD:C_0805_2012Metric_Pad1.18x1.45mm_HandSolder
- C8: renamed from C10; footprint (none) -> Capacitor_SMD:C_0805_2012Metric_Pad1.18x1.45mm_HandSolder
- C9: renamed from C2; footprint (none) -> Capacitor_SMD:C_0805_2012Metric_Pad1.18x1.45mm_HandSolder
- J1: footprint (none) -> Connector_Audio:Jack_3.5mm_Lumberg_1503_02_Horizontal
- R1: renamed from R5; footprint (none) -> Resistor_SMD:R_0805_2012Metric_Pad1.20x1.40mm_HandSolder
- R10, R11, R12, R13, R14, R15, R16, R17, R18, R7, R8, R9, RV1, RV2: footprint (none) -> Resistor_SMD:R_0805_2012Metric_Pad1.20x1.40mm_HandSolder
- R2: renamed from R6; footprint (none) -> Resistor_SMD:R_0805_2012Metric_Pad1.20x1.40mm_HandSolder
- R3: renamed from R1; footprint (none) -> Resistor_SMD:R_0805_2012Metric_Pad1.20x1.40mm_HandSolder
- R4: renamed from R2; footprint (none) -> Resistor_SMD:R_0805_2012Metric_Pad1.20x1.40mm_HandSolder
- R5: renamed from R3; footprint (none) -> Resistor_SMD:R_0805_2012Metric_Pad1.20x1.40mm_HandSolder
- R6: renamed from R4; footprint (none) -> Resistor_SMD:R_0805_2012Metric_Pad1.20x1.40mm_HandSolder
- SW1: renamed from SW3; footprint (none) -> Rotary_Encoder:RotaryEncoder_Alps_EC12E-Switch_Vertical_H20mm
- SW2: renamed from SW4; footprint (none) -> Rotary_Encoder:RotaryEncoder_Alps_EC12E-Switch_Vertical_H20mm
- SW3: renamed from SW1; footprint (none) -> Button_Switch_THT:SW_PUSH_6mm
- SW4: renamed from SW5; footprint (none) -> Rotary_Encoder:RotaryEncoder_Alps_EC12E-Switch_Vertical_H20mm
- SW5: renamed from SW2; footprint (none) -> Button_Switch_THT:SW_PUSH_6mm
- TP1, TP10, TP11, TP12, TP2, TP3, TP4, TP5, TP6, TP7, TP8, TP9: footprint (none) -> Library:TouchPad_D12mm
- renumbered U2 to U1, U3 to U2, U1 to U3

Commit message: Added all footprints / Made v1 of the PCB
Parts:
- RV1, RV2: footprint Resistor_SMD:R_0805_2012Metric_Pad1.20x1.40mm_HandSolder -> Potentiometer_THT:Potentiometer_Alps_RK09K_Single_Vertical
Other:
- note added: "Fuji Synth v1.0"
Changed lines of the file:
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@@
 		)
 	)
+	(text "Fuji Synth v1.0"
+		(exclude_from_sim no)
+		(at 211.836 18.796 0)
+		(effects
+			(font
+				(size 2.54 2.54)
+				(thickness 0.508)
+				(bold yes)
+			)
+		)
+	)
 	(text "3x Rotary Encoder (SW3,4,5)"
 		(exclude_from_sim no)
@@
 			)
 		)
-		(property "Footprint" "Resistor_SMD:R_0805_2012Metric_Pad1.20x1.40mm_HandSolder"
+		(property "Footprint" "Potentiometer_THT:Potentiometer_Alps_RK09K_Single_Vertical"
 			(at 191.77 123.19 0)
 			(hide yes)
@@
 			)
 		)
-		(property "Footprint" "Resistor_SMD:R_0805_2012Metric_Pad1.20x1.40mm_HandSolder"
+		(property "Footprint" "Potentiometer_THT:Potentiometer_Alps_RK09K_Single_Vertical"
 			(at 160.02 123.19 0)
 			(hide yes)

Commit message: PCB version 2 / removed old gerber files
Parts:
- added H1, H2, H3, H4: MountingHole, MountingHole:MountingHole_2.2mm_M2, symbol Mechanical:MountingHole

Commit message: New potentiometers / Finished routing v1
Parts:
- RV1, RV2: footprint Potentiometer_THT:Potentiometer_Alps_RK09K_Single_Vertical -> Potentiometer_THT:Potentiometer_Bourns_PTA1543_Single_Slide
Changed lines of the file:
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@@
 			)
 		)
-		(property "Footprint" "Potentiometer_THT:Potentiometer_Alps_RK09K_Single_Vertical"
+		(property "Footprint" "Potentiometer_THT:Potentiometer_Bourns_PTA1543_Single_Slide"
 			(at 191.77 123.19 0)
 			(hide yes)
@@
 			)
 		)
-		(property "Footprint" "Potentiometer_THT:Potentiometer_Alps_RK09K_Single_Vertical"
+		(property "Footprint" "Potentiometer_THT:Potentiometer_Bourns_PTA1543_Single_Slide"
 			(at 160.02 123.19 0)
 			(hide yes)

Commit message: New files / new wiring / started the firmware
Other:
- note added: "2x Buttons (SW3,5)"
- note added: "3x Rotary Encoder (SW1,2,4)"
- note added: "MPR121 (U3)"
- note added: "OLED (U2)"
- note added: "PCM5102A + Jack (U1) (J1)"
- note removed: "2x Buttons (SW1,2)"
- note removed: "3x Rotary Encoder (SW3,4,5)"
- note removed: "MPR121 (U1)"
- note removed: "OLED (U3)"
- note removed: "PCM5102A + Jack (U2) (J1)"
Changed lines of the file:
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@@
 		)
 	)
-	(text "OLED (U3)"
+	(text "OLED (U2)"
 		(exclude_from_sim no)
 		(at 100.838 167.386 0)
@@
 		)
 	)
-	(text "PCM5102A + Jack (U2) (J1)"
+	(text "PCM5102A + Jack (U1) (J1)"
 		(exclude_from_sim no)
 		(at 41.148 178.054 0)
@@
 		)
 	)
-	(text "2x Buttons (SW1,2)"
+	(text "2x Buttons (SW3,5)"
 		(exclude_from_sim no)
 		(at 167.894 163.83 0)
@@
 		)
 	)
-	(text "MPR121 (U1)"
+	(text "MPR121 (U3)"
 		(exclude_from_sim no)
 		(at 119.634 74.168 0)
@@
 		)
 	)
-	(text "3x Rotary Encoder (SW3,4,5)"
+	(text "3x Rotary Encoder (SW1,2,4)"
 		(exclude_from_sim no)
 		(at 133.35 109.22 0)
@@
 	)
 	(junction
-		(at 54.61 20.32)
-		(diameter 0)
-		(color 0 0 0 0)
-	)
-	(junction
-		(at 55.88 133.35)
-		(diameter 0)
-		(color 0 0 0 0)
-	)
-	(junction
-		(at 59.69 20.32)
-		(diameter 0)
-		(color 0 0 0 0)
-	)
-	(junction
 		(at 148.59 102.87)
 		(diameter 0)
@@
 	)
 	(junction
+		(at 55.88 133.35)
+		(diameter 0)
+		(color 0 0 0 0)
+	)
+	(junction
 		(at 73.66 160.02)
 		(diameter 0)
@@
 	(wire
 		(pts
-			(xy 60.96 20.32) (xy 59.69 20.32)
-		)
-		(stroke
-			(width 0)
-			(type default)
-		)
-	)
-	(wire
-		(pts
-			(xy 54.61 20.32) (xy 54.61 24.13)
+			(xy 54.61 19.05) (xy 54.61 24.13)
 		)
 		(stroke
@@
 	(wire
 		(pts
-			(xy 59.69 20.32) (xy 59.69 24.13)
+			(xy 59.69 19.05) (xy 59.69 24.13)
 		)
 		(stroke
@@
 	(wire
 		(pts
-			(xy 167.64 43.18) (xy 165.1 43.18)
+			(xy 55.88 130.81) (xy 55.88 133.35)
 		)
 		(stroke
@@
 	(wire
 		(pts
-			(xy 74.93 120.65) (xy 74.93 121.92)
+			(xy 167.64 43.18) (xy 165.1 43.18)
 		)
 		(stroke
@@
 	(wire
 		(pts
-			(xy 109.22 95.25) (xy 109.22 105.41)
+			(xy 74.93 120.65) (xy 74.93 121.92)
 		)
 		(stroke
@@
 	(wire
 		(pts
-			(xy 53.34 20.32) (xy 54.61 20.32)
+			(xy 109.22 95.25) (xy 109.22 105.41)
 		)
 		(stroke
@@
 	(wire
 		(pts
-			(xy 59.69 19.05) (xy 59.69 20.32)
-		)
-		(stroke
-			(width 0)
-			(type default)
-		)
-	)
-	(wire
-		(pts
 			(xy 30.48 69.85) (xy 31.75 69.85)
 		)
@@
 	(wire
 		(pts
-			(xy 54.61 19.05) (xy 54.61 20.32)
-		)
-		(stroke
-			(width 0)
-			(type default)
-		)
-	)
-	(wire
-		(pts
 			(xy 191.77 134.62) (xy 189.23 134.62)
 		)
@@
 	(symbol
 		(lib_id "power:PWR_FLAG")
-		(at 55.88 133.35 0)
+		(at 55.88 130.81 0)
 		(unit 1)
 		(body_style 1)
@@
 		(fields_autoplaced yes)
 		(property "Reference" "#FLG01"
-			(at 55.88 131.445 0)
+			(at 55.88 128.905 0)
 			(hide yes)
 			(show_name no)
@@
 		)
 		(property "Value" "PWR_FLAG"
-			(at 55.88 128.27 0)
+			(at 55.88 125.73 0)
 			(show_name no)
 			(do_not_autoplace no)
@@
 		)
 		(property "Footprint" ""
-			(at 55.88 133.35 0)
+			(at 55.88 130.81 0)
 			(hide yes)
 			(show_name no)
@@
 		)
 		(property "Datasheet" ""
-			(at 55.88 133.35 0)
+			(at 55.88 130.81 0)
 			(hide yes)
 			(show_name no)
@@
 		)
 		(property "Description" "Special symbol for telling ERC where power comes from"
-			(at 55.88 133.35 0)
+			(at 55.88 130.81 0)
 			(hide yes)
 			(show_name no)
