File: Fuji-Synth/Fuji-Synth.kicad_pcb (KiCad board)
At the start: 2 copper layers, 135.5 x 82.4 mm, 58 parts, among them J1 AudioJack3, SW1 RotaryEncoder_Switch, SW2 RotaryEncoder_Switch, SW3 SW_Push, SW4 RotaryEncoder_Switch, SW5 SW_Push, U1 PCM5102A, U2 ER_OLEDM0.91_1x-I2C, U3 MPR121QR2

Commit message: PCB version 2 / removed old gerber files
Parts:
- moved H1 151.9 mm to (169.9, 55.5), turned to 180 degrees
- moved H3 138.4 mm to (75.2, 55.5), turned to 180 degrees
- moved C12 125.3 mm to (169.7, 100.1), turned to 90 degrees
- moved C3 87.6 mm to (83.8, 94.5)
- moved C7 75.8 mm to (87.9, 89.9), turned to 0 degrees
- moved RV1 75.1 mm to (98.0, 73.2), turned to -90 degrees
- moved C9 68.5 mm to (99.0, 95.0), turned to 0 degrees
- moved C8 67.0 mm to (130.6, 94.5)
- moved C11 65.4 mm to (91.4, 94.5), turned to 0 degrees
- moved C2 64.7 mm to (169.2, 117.3), turned to 90 degrees
- moved TP11 62.5 mm to (132.7, 125.1)
- moved C10 62.5 mm to (169.1, 141.7), turned to 0 degrees
- moved R14 62.2 mm to (124.1, 132.2)
- moved TP8 61.4 mm to (116.8, 125.2)
- moved R11 61.4 mm to (108.4, 132.2)
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Other:
- board size 135.5 x 82.4 mm -> 100 x 100 mm

Commit message: New potentiometers / Finished routing v1
Parts:
- RV1, RV2: footprint Potentiometer_THT:Potentiometer_Alps_RK09K_Single_Vertical -> Potentiometer_THT:Potentiometer_Bourns_PTA1543_Single_Slide
- moved C7 36.5 mm to (124.0, 95.0)
- moved RV2 20.6 mm to (103.0, 76.8), turned to 180 degrees
- moved RV1 16.7 mm to (103.2, 89.1), turned to 180 degrees
- moved C3 6.80 mm to (78.0, 98.0)
- moved C11 2.74 mm to (92.5, 97.0)
- moved U3 1.39 mm to (108.0, 96.0)
- moved R13 1.22 mm to (124.0, 115.0)
- moved SW4 1.15 mm to (125.7, 77.8)
- moved SW2 1.15 mm to (107.0, 77.8)
- moved C9 1.02 mm to (99.0, 96.0)
- moved U2 0.62 mm to (102.5, 64.8)
- moved R10 0.35 mm to (108.0, 114.4)
- moved SW1 0.25 mm to (81.7, 58.5)
Routing:
- net GND: track 0.00 -> 632.0 mm, vias 0 -> 14
- net I2C_SDA: track 0.00 -> 365.7 mm, vias 0 -> 3
- net +3V3: track 0.00 -> 307.8 mm, vias 0 -> 7
- net TOUCH_IRQ: track 0.00 -> 233.6 mm, vias 0 -> 5
- net POT_PITCH: track 0.00 -> 141.7 mm
- net I2C_SCL: track 0.00 -> 136.5 mm, vias 0 -> 6
- net Net-(U3-LED7/ELE11): track 0.00 -> 130.7 mm, vias 0 -> 2
- net Net-(A1-ADC_VREF): track 0.00 -> 124.6 mm, vias 0 -> 4
- net POT_FILTER: track 0.00 -> 121.8 mm
- net ENC1_B: track 0.00 -> 119.9 mm
- net Net-(U3-LED3/ELE7): track 0.00 -> 117.4 mm, vias 0 -> 3
- net Net-(U3-ELE2): track 0.00 -> 108.6 mm, vias 0 -> 2
- net ENC1_SW: track 0.00 -> 108.0 mm, vias 0 -> 2
- net ENC1_A: track 0.00 -> 103.1 mm, vias 0 -> 1
- net ENC3_A: track 0.00 -> 92.8 mm, vias 0 -> 3
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
Commit message: New gerbers / Pcb v2.1 / Cad files for knobs
Routing:
- net Net-(U3-LED3/ELE7): track 117.4 -> 52.5 mm, vias 3 -> 2
- net I2S_BCK: track 55.8 -> 80.0 mm
- net ENC1_A: track 103.1 -> 127.0 mm
- net TOUCH_IRQ: track 233.6 -> 248.7 mm
- net Net-(A1-ADC_VREF): track 124.6 -> 135.7 mm
- net ENC3_B: track 51.3 -> 59.8 mm
- net Net-(U3-LED2/ELE6): track 28.8 -> 36.8 mm
- net Net-(U3-LED7/ELE11): track 130.7 -> 137.0 mm
- net I2S_LRCK: track 59.9 -> 53.7 mm
- net GND: track 632.0 -> 637.7 mm
- net +3V3: track 307.8 -> 312.6 mm
- net Net-(U3-ELE1): track 50.3 -> 54.7 mm
- net Net-(U1-OUTR): track 43.7 -> 47.6 mm
- net Net-(U3-LED0/ELE4): track 50.8 -> 47.2 mm
- net ENC1_SW: track 108.0 -> 111.1 mm
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
Commit message: Pcb routing updated / new new gerbers again
Parts:
- added G***: LOGO, LOGO, F.Cu at (75.8, 117.1)
Routing:
- net BTN1: track 59.4 -> 446.6 mm
- net OUT_L: track 27.0 -> 18.3 mm
- net I2C_SCL: track 136.5 -> 131.2 mm
- net ENC3_A: track 93.6 -> 88.5 mm
- net ENC1_B: track 119.9 -> 115.2 mm
- net TOUCH_IRQ: track 248.7 -> 244.4 mm
- net +3V3: track 312.6 -> 308.7 mm
- net Net-(U3-LED4/ELE8): track 69.4 -> 72.5 mm
- net POT_PITCH: track 141.8 -> 144.7 mm
- net Net-(U3-LED2/ELE6): track 36.8 -> 39.7 mm
- net I2S_DOUT: track 85.8 -> 88.3 mm
- net I2C_SDA: track 366.3 -> 368.6 mm
- net Net-(U3-LED3/ELE7): track 52.5 -> 54.6 mm
- net Net-(U3-ELE3): track 26.7 -> 28.5 mm
- net ENC1_A: track 127.0 -> 128.6 mm
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Other:
- board text added: "@A41K"
- board text added: "Fuji Synth"
- board text added: "v1.0"

Commit message: New files / new wiring / started the firmware
Parts:
- moved G*** 0.34 mm to (75.5, 117.1)
Routing:
- net BTN1: track 446.6 -> 165.1 mm
- net I2C_SDA: track 368.6 -> 276.2 mm, vias 3 -> 2
- net I2S_DOUT: track 88.3 -> 120.6 mm
- net TOUCH_IRQ: track 244.4 -> 234.0 mm
- net GND: track 638.2 -> 627.9 mm
- net Net-(U1-OUTR): track 47.6 -> 39.6 mm
- net ENC1_B: track 115.2 -> 108.1 mm
- net ENC1_SW: track 109.6 -> 103.2 mm
- net Net-(U3-ELE2): track 106.5 -> 102.5 mm
- net I2S_BCK: track 80.0 -> 76.9 mm
- net +3V3: track 308.7 -> 305.6 mm
- net Net-(U3-ELE3): track 28.5 -> 25.8 mm
- net POT_PITCH: track 144.7 -> 142.4 mm
- net Net-(U1-OUTL): track 18.2 -> 16.2 mm
- net ENC1_A: track 128.6 -> 127.0 mm
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
Commit message: Some wiring fixing / half firmware done
Routing:
- net BTN1: track 165.1 -> 83.4 mm
- net Net-(A1-ADC_VREF): track 136.6 -> 126.0 mm
- net ENC1_A: track 127.0 -> 119.7 mm
- net TOUCH_IRQ: track 234.0 -> 227.2 mm
- net ENC1_B: track 108.1 -> 101.7 mm
- net POT_PITCH: track 142.4 -> 138.6 mm
- net Net-(U3-ELE0): track 36.0 -> 32.3 mm
- net ENC2_B: track 57.4 -> 54.5 mm
- net GND: track 627.9 -> 625.2 mm
- net I2S_DOUT: track 120.6 -> 119.2 mm
- net Net-(U3-ELE2): track 102.5 -> 101.2 mm
- net ENC3_A: track 88.5 -> 87.3 mm
- net Net-(U3-ELE1): track 54.0 -> 55.1 mm
- net ENC2_SW: track 60.2 -> 59.3 mm
- net Net-(U3-LED1/ELE5): track 63.1 -> 62.6 mm
